File: KiCAD/seq.kicad_pcb (KiCad board)
At the start: 2 copper layers, 31 parts, among them P1 CONN_01X03, P2 CONN_01X02, P3 CONN_01X08, U1 cd4016, U2 cd4016

Commit message: esquema errado
Parts:
- moved P2 93.8 mm to (139.2, 115.3)
- moved R1 31.1 mm to (134.6, 47.6), turned to 270 degrees
- moved R7 30.3 mm to (91.0, 70.1), turned to 0 degrees
- moved RV5 22.5 mm to (132.1, 118.1), turned to 270 degrees
- moved R6 21.0 mm to (101.2, 96.1), turned to 0 degrees
- moved RV7 20.4 mm to (90.2, 86.4), turned to 180 degrees
- moved RV6 18.2 mm to (104.5, 110.9), turned to 225 degrees
- moved R8 18.1 mm to (110.9, 53.6)
- moved R3 18.0 mm to (162.6, 91.4)
- moved D7 17.3 mm to (96.5, 81.3), turned to 180 degrees
- moved C1 16.8 mm to (149.9, 71.8)
- moved D5 15.9 mm to (127.0, 111.8), turned to 270 degrees
- moved R2 15.3 mm to (152.4, 66.0)
- moved C2 15.1 mm to (103.5, 89.8), turned to 180 degrees
- moved D4 14.5 mm to (148.6, 102.8), turned to 315 degrees
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Routing:
- net cvout: track 0.00 -> 245.1 mm
- net +5V: track 27.4 -> 169.8 mm
- net Net-(P3-Pad5): track 154.8 -> 56.7 mm, vias 0 -> 2
- net Net-(RV8-Pad1): track 97.6 -> 40.8 mm
- net Net-(RV3-Pad1): track 0.00 -> 55.8 mm, vias 0 -> 2
- net Net-(RV1-Pad1): track 0.00 -> 50.4 mm
- net Net-(P3-Pad1): track 0.00 -> 48.3 mm, vias 0 -> 2
- net Net-(P3-Pad2): track 0.00 -> 44.1 mm
- net Net-(P3-Pad3): track 0.00 -> 43.4 mm
- net Net-(RV2-Pad1): track 0.00 -> 35.6 mm, vias 0 -> 2
- net Net-(RV4-Pad1): track 0.00 -> 29.1 mm
- net Net-(P3-Pad4): track 0.00 -> 28.1 mm, vias 0 -> 2
- net Net-(RV5-Pad1): track 71.1 -> 51.4 mm
- net Net-(D3-Pad2): track 0.00 -> 11.2 mm
- net Net-(D8-Pad2): track 18.6 -> 9.02 mm
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- added copper zone on B.Cu, net GND
Other:
- board outline added: 96 x 93.5 mm
