File: KiCAD/seq.sch (KiCad schematic (older format))
At the start: 31 parts, among them P1 CONN_01X03, P2 CONN_01X02, P3 CONN_01X08, U1 cd4016, U2 cd4016

Commit message: updated schematic
added arduino mini and simple 5V power supply to the schematic. my
library also updated with arduino mini schematic.
Parts:
- removed P1: CONN_01X03, Pin_Headers:Pin_Header_Straight_1x03, symbol CONN_01X03
- removed P2: CONN_01X02, Pin_Headers:Pin_Header_Straight_1x02, symbol CONN_01X02
- removed P3: CONN_01X08, Pin_Headers:Pin_Header_Straight_1x08, symbol CONN_01X08
- removed RV1, RV2, RV3, RV4, RV5, RV6, RV7, RV8: 100k, Potentiometers:Potentiometer_WirePads_largePads, symbol POT
- added C? (x2): CP, symbol CP
- added C? (x2): C, symbol C
- added P?: CONN_01X03, symbol CONN_01X03
- added P?: CONN_02X05, symbol CONN_02X05
- added RV? (x8): 100k, symbol POT
- added RV?: 10k, symbol POT
- added U?: 78L05, symbol 78L05
- added uC?: arduino_mini_pro, symbol arduino_mini_pro
- D1, D2, D3, D4, D5, D6, D7, D8: symbol LED -> LED-RESCUE-seq
Connections:
- net labels added: +12V, -12V, gate
- wire segments 103 -> 105
- no-connect marks 0 -> 11
Other:
- moved on the sheet: C1, C2, D1, D2, D3, D4, D5, D6, D7, D8, R1, R2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
